Commit message: Fix scale errors in meshes and adjust positions of links and joints in the urdf

File: reachy.URDF (robot description, URDF)
Before this commit: robot Reachy, 20 links, 19 joints
Links:
- link l_shoulder_x: geometry collision mesh filename=package://reachy_description/meshes/shoulder_x.dae; visual mesh filename=package://reachy_description/meshes/shoulder_x.dae
- link r_shoulder_x: geometry collision mesh filename=package://reachy_description/meshes/shoulder_x.dae; visual mesh filename=package://reachy_description/meshes/shoulder_x.dae
Joints:
- joint l_antenna: origin xyz=-0.052 0.057 0.086 rpy=9.52078 -60.4 -63.6 -> xyz=-0.052 0.057 0.086 rpy=0.166 -1.054 -1.11
- joint l_gripper: origin xyz=0 -0.01 -0.075 rpy=0.0 0.0 0.0 -> xyz=0.0 0.037 -0.03998 rpy=0.0 0.0 0.0
- joint r_antenna: origin xyz=-0.052 -0.057 0.086 rpy=-9.52078 -60.4 63.6 -> xyz=-0.052 -0.057 0.086 rpy=-0.166 -1.054 1.11
- joint r_gripper: origin xyz=0 -0.01 -0.075 rpy=0.0 0.0 0.0 -> xyz=0.0 -0.037 -0.03998 rpy=0.0 0.0 0.0

Commit message: Update limits of joints and the location of the head in the urdf

File: reachy.URDF (robot description, URDF)
Before this commit: robot Reachy, 20 links, 19 joints
Joints:
- joint l_elbow_pitch: limit lower=0 upper=2.182 effort=10. velocity=0.0 -> lower=-2.182 upper=0 effort=10. velocity=0.0
- joint l_forearm_yaw: limit lower=-1.175 upper=1.175 effort=10. velocity=0.0 -> lower=-1.745 upper=1.745 effort=10. velocity=0.0
- joint l_shoulder_pitch: limit lower=-1.0412 upper=3.14 effort=10. velocity=0.0 -> lower=-2.618 upper=1.57 effort=10. velocity=0.0
- joint l_shoulder_roll: limit lower=-1.57 upper=1.745 effort=10. velocity=0.0 -> lower=-0.174 upper=3.14 effort=10. velocity=0.0
- joint r_elbow_pitch: limit lower=0 upper=2.182 effort=10. velocity=0.0 -> lower=-2.182 upper=0 effort=10. velocity=0.0
- joint r_forearm_yaw: limit lower=-1.175 upper=1.175 effort=10. velocity=0.0 -> lower=-1.745 upper=1.745 effort=10. velocity=0.0
- joint r_shoulder_pitch: limit lower=-3.14 upper=1.0412 effort=10. velocity=0.0 -> lower=-2.618 upper=1.57 effort=10. velocity=0.0
- joint r_shoulder_roll: limit lower=-1.745 upper=1.57 effort=10. velocity=0.0 -> lower=-3.14 upper=0.174 effort=10. velocity=0.0
- joint torso2head: origin xyz=0 0 0.25 rpy=0 0 0 -> xyz=0.015 0.0 0.095 rpy=0 0.174 0

Commit message: Added collision model

File: reachy.URDF (robot description, URDF)
Before this commit: robot Reachy, 20 links, 19 joints
Links:
- link head: geometry collision cylinder length=0.15 radius=0.06; visual mesh filename=package://reachy_description/meshes/head.dae
- link l_antenna: geometry visual mesh filename=package://reachy_description/meshes/antenna.dae
- link l_forearm: geometry collision cylinder length=0.09 radius=0.04; visual mesh filename=package://reachy_description/meshes/forearm.dae
- link l_gripper_finger: geometry collision box size=0.1 0.012 0.035; visual mesh filename=package://reachy_description/meshes/l_gripper_finger.dae
- link l_gripper_thumb: geometry collision box size=0.1 0.012 0.035; visual mesh filename=package://reachy_description/meshes/l_gripper_thumb.dae
- link l_shoulder: geometry collision cylinder length=0.09 radius=0.035; visual mesh filename=package://reachy_description/meshes/shoulder.dae
- link l_shoulder_x: geometry collision cylinder length=0.04 radius=0.035; visual mesh filename=package://reachy_description/meshes/shoulder_x.dae
- link l_upper_arm: geometry collision cylinder length=0.25 radius=0.04; visual mesh filename=package://reachy_description/meshes/upper_arm.dae
- link l_wrist: geometry collision cylinder length=0.14 radius=0.035; visual mesh filename=package://reachy_description/meshes/wrist.dae
- link l_wrist2hand: geometry collision cylinder length=0.06 radius=0.03; visual mesh filename=package://reachy_description/meshes/wrist2hand.dae
- link r_antenna: geometry visual cylinder length=0.15 radius=0.005
- link r_forearm: geometry collision cylinder length=0.09 radius=0.04; visual mesh filename=package://reachy_description/meshes/forearm.dae
- link r_gripper_finger: geometry collision box size=0.1 0.012 0.035; visual mesh filename=package://reachy_description/meshes/r_gripper_finger.dae
- link r_gripper_thumb: geometry collision box size=0.1 0.012 0.035; visual mesh filename=package://reachy_description/meshes/r_gripper_thumb.dae
- link r_shoulder: geometry collision cylinder length=0.09 radius=0.035; visual mesh filename=package://reachy_description/meshes/shoulder.dae
- link r_shoulder_x: geometry collision cylinder length=0.04 radius=0.035; visual mesh filename=package://reachy_description/meshes/shoulder_x.dae
- link r_upper_arm: geometry collision cylinder length=0.25 radius=0.04; visual mesh filename=package://reachy_description/meshes/upper_arm.dae
- link r_wrist: geometry collision cylinder length=0.14 radius=0.035; visual mesh filename=package://reachy_description/meshes/wrist.dae
- link r_wrist2hand: geometry collision cylinder length=0.06 radius=0.03; visual mesh filename=package://reachy_description/meshes/wrist2hand.dae
- link torso: geometry collision box size=0.11 0.2 0.32; visual mesh filename=package://reachy_description/meshes/torso.dae

Commit message: Fix left antenna

File: reachy.URDF (robot description, URDF)
Before this commit: robot reachy, 20 links, 19 joints
Links:
- link r_antenna: geometry visual mesh filename=package://reachy_description/meshes/antenna.dae

Commit message: Added pedestal and tips

File: reachy.URDF (robot description, URDF)
Before this commit: robot reachy, 20 links, 19 joints
Links:
- added link left_tip
- added link pedestal
- added link right_tip
Joints:
- added joint l_tip: type fixed, parent l_gripper_finger, child left_tip, origin xyz=0 -0.025 -0.045 rpy=0 0 0
- added joint pedestal: type fixed, parent pedestal, child torso, origin xyz=0 0 1 rpy=0 0 0
- added joint r_tip: type fixed, parent r_gripper_finger, child right_tip, origin xyz=0 0.025 -0.045 rpy=0 0 0

Commit message: Fixed kinematic chains to tips

File: reachy.URDF (robot description, URDF)
Before this commit: robot reachy, 23 links, 22 joints
Joints:
- joint l_tip: origin xyz=0 -0.025 -0.045 rpy=0 0 0 -> xyz=0 0.012 -0.085 rpy=0 0 0; parent l_gripper_finger -> l_gripper_thumb
- joint r_tip: origin xyz=0 0.025 -0.045 rpy=0 0 0 -> xyz=0 -0.012 -0.085 rpy=0 0 0; parent r_gripper_finger -> r_gripper_thumb

Commit message: Head ball joint

File: reachy.URDF (robot description, URDF)
Before this commit: robot reachy, 23 links, 22 joints
Links:
- added link head_x
- added link head_y
Joints:
- removed joint torso2head
- added joint head_pitch: type revolute, parent head_x, child head_y, origin xyz=0 0 0 rpy=0.0 0.0 0.0, axis 0 1 0, limit lower=0 upper=0.8 effort=10. velocity=0.0
- added joint head_roll: type revolute, parent torso, child head_x, origin xyz=0.015 0.0 0.095 rpy=0 0.174 0, axis 1 0 0, limit lower=0 upper=0.8 effort=10. velocity=0.0
- added joint head_yaw: type revolute, parent head_y, child head, origin xyz=0 0 0 rpy=0.0 0.0 0.0, axis 0 0 1, limit lower=0 upper=0.8 effort=10. velocity=0.0

Commit message: Oribta renaming + additional fixed link

File: reachy.URDF (robot description, URDF)
Before this commit: robot reachy, 25 links, 24 joints
Links:
- added link head_z
Joints:
- removed joint head_pitch
- removed joint head_roll
- removed joint head_yaw
- added joint orbita_fixed: type fixed, parent head_z, child head, origin xyz=0 0 0 rpy=0.0 0.0 0.0
- added joint orbita_pitch: type revolute, parent head_x, child head_y, origin xyz=0 0 0 rpy=0.0 0.0 0.0, axis 0 1 0, limit lower=0 upper=0.8 effort=10. velocity=0.0
- added joint orbita_roll: type revolute, parent torso, child head_x, origin xyz=0.015 0.0 0.095 rpy=0 0.174 0, axis 1 0 0, limit lower=0 upper=0.8 effort=10. velocity=0.0
- added joint orbita_yaw: type revolute, parent head_y, child head_z, origin xyz=0 0 0 rpy=0.0 0.0 0.0, axis 0 0 1, limit lower=-0.8 upper=0.8 effort=10. velocity=0.0

Commit message: Camera links

File: reachy.URDF (robot description, URDF)
Before this commit: robot reachy, 26 links, 25 joints
Links:
- added link left_camera
- added link right_camera
Joints:
- added joint left_cam_fixed: type fixed, parent head, child left_camera, origin xyz=0 0.04 0.06 rpy=0.0 0.0 0.0
- added joint right_cam_fixed: type fixed, parent head, child right_camera, origin xyz=0 -0.04 0.06 rpy=0.0 0.0 0.0

Commit message: Add meshes and visual for orbita

File: reachy.URDF (robot description, URDF)
Before this commit: robot reachy, 28 links, 27 joints
Links:
- link head_x: geometry visual mesh filename=package://reachy_description/meshes/orbita_arm.dae
- link head_y: geometry visual mesh filename=package://reachy_description/meshes/orbita_arm.dae
- link head_z: geometry visual mesh filename=package://reachy_description/meshes/orbita_arm.dae

Commit message: Adjust the position of cameras joints

File: reachy.URDF (robot description, URDF)
Before this commit: robot reachy, 28 links, 27 joints
Joints:
- joint left_cam_fixed: origin xyz=0 0.04 0.06 rpy=0.0 0.0 0.0 -> xyz=0.0033 0.03625 0.061 rpy=0.0 0.0 0.0
- joint right_cam_fixed: origin xyz=0 -0.04 0.06 rpy=0.0 0.0 0.0 -> xyz=0.0033 -0.03625 0.061 rpy=0.0 0.0 0.0

Commit message: Add fixed joints and links to fix the arms of Orbita

File: reachy.URDF (robot description, URDF)
Before this commit: robot reachy, 28 links, 27 joints
Links:
- added link bottom_arm; visual mesh filename=package://reachy_description/meshes/orbita_arm.dae
- added link middle_arm; visual mesh filename=package://reachy_description/meshes/orbita_arm.dae
- added link top_arm; visual mesh filename=package://reachy_description/meshes/orbita_arm.dae
- link head_x: geometry 
- link head_y: geometry 
- link head_z: geometry 
Joints:
- added joint orbita_bottom: type fixed, parent torso, child bottom_arm, origin xyz=0.0067 0.0 0.0478 rpy=0 0.174 0
- added joint orbita_middle: type fixed, parent torso, child middle_arm, origin xyz=0.0067 0.0 0.0478 rpy=0 0.174 0
- added joint orbita_top: type fixed, parent torso, child top_arm, origin xyz=0.0067 0.0 0.0478 rpy=0 0.174 0

Commit message: Adjust Roll-Pitch-Yaw angles limits of the head

File: reachy.URDF (robot description, URDF)
Before this commit: robot reachy, 31 links, 30 joints
Joints:
- joint orbita_pitch: limit lower=0 upper=0.8 effort=10. velocity=0.0 -> lower=-0.8 upper=1.13 effort=10. velocity=0.0
- joint orbita_roll: limit lower=0 upper=0.8 effort=10. velocity=0.0 -> lower=-0.8 upper=0.8 effort=10. velocity=0.0
- joint orbita_yaw: limit lower=-0.8 upper=0.8 effort=10. velocity=0.0 -> lower=-2.79 upper=2.79 effort=10. velocity=0.0

Commit message: Empty collisions for Orbita and Antennas

File: reachy.URDF (robot description, URDF)
Before this commit: robot reachy, 31 links, 30 joints
Links:
- removed link bottom_arm
- removed link middle_arm
- removed link top_arm
- added link bottom_orbita_arm; collision cylinder length=0.0 radius=0.0; visual mesh filename=package://reachy_description/meshes/orbita_arm.dae
- added link middle_orbita_arm; collision cylinder length=0.0 radius=0.0; visual mesh filename=package://reachy_description/meshes/orbita_arm.dae
- added link top_orbita_arm; collision cylinder length=0.0 radius=0.0; visual mesh filename=package://reachy_description/meshes/orbita_arm.dae
- link l_antenna: geometry collision cylinder length=0.0 radius=0.0; visual mesh filename=package://reachy_description/meshes/antenna.dae
- link r_antenna: geometry collision cylinder length=0.0 radius=0.0; visual mesh filename=package://reachy_description/meshes/antenna.dae
Joints:
- joint orbita_bottom: child bottom_arm -> bottom_orbita_arm
- joint orbita_middle: child middle_arm -> middle_orbita_arm
- joint orbita_top: child top_arm -> top_orbita_arm
